File: Arduino-MotionSensors.sch (KiCad schematic (older format))
At the start: 22 parts

Commit message: Renamed files to match upper folder, adjusted for ERC issues, added initial Arduino sketch.
Parts:
- gave numbers to parts that had none: 22
Connections:
- net +5V: now also IC1.20 (AVCC), IC1.7 (VCC)
Changed lines of the file:
@@
 LIBS:contrib
 LIBS:valves
-LIBS:MotionSensorLights-cache
+LIBS:Arduino-MotionSensors-cache
 EELAYER 27 0
 EELAYER END
@@
 $EndComp
 $Comp
-L DIODE D?
+L DIODE D1
 U 1 1 531C655B
 P 1300 750
-F 0 "D?" H 1300 850 40  0000 C CNN
+F 0 "D1" H 1300 850 40  0000 C CNN
 F 1 "1N4007" H 1300 650 40  0000 C CNN
 F 2 "~" H 1300 750 60  0000 C CNN
@@
 $EndComp
 $Comp
-L CP1 C?
+L CP1 C1
 U 1 1 531C66B9
 P 1650 950
-F 0 "C?" H 1700 1050 50  0000 L CNN
+F 0 "C1" H 1700 1050 50  0000 L CNN
 F 1 "470uF" H 1700 850 50  0000 L CNN
 F 2 "~" H 1650 950 60  0000 C CNN
@@
 $EndComp
 $Comp
-L CP1 C?
+L CP1 C2
 U 1 1 531C67A5
 P 2800 950
-F 0 "C?" H 2850 1050 50  0000 L CNN
+F 0 "C2" H 2850 1050 50  0000 L CNN
 F 1 "1uF" H 2850 850 50  0000 L CNN
 F 2 "~" H 2800 950 60  0000 C CNN
@@
 $EndComp
 $Comp
-L LM7805CT U?
+L LM7805CT U1
 U 1 1 531C6864
 P 2250 800
-F 0 "U?" H 2050 1000 40  0000 C CNN
+F 0 "U1" H 2050 1000 40  0000 C CNN
 F 1 "LM7805CT" H 2250 1000 40  0000 L CNN
 F 2 "TO-220" H 2250 900 30  0000 C CIN
@@
 Connection ~ 2250 1150
 $Comp
-L ATMEGA328-P IC?
+L ATMEGA328-P IC1
 U 1 1 531C6BF5
 P 4750 3250
-F 0 "IC?" H 4000 4500 40  0000 L BNN
+F 0 "IC1" H 4000 4500 40  0000 L BNN
 F 1 "ATMEGA328-P" H 5150 1850 40  0000 L BNN
 F 2 "DIL28" H 4750 3250 30  0000 C CIN
@@
 	3850 4450 3850 4350
 $Comp
-L CRYSTAL X?
+L CRYSTAL X1
 U 1 1 531C78FA
 P 7850 2700
-F 0 "X?" H 7850 2850 60  0000 C CNN
+F 0 "X1" H 7850 2850 60  0000 C CNN
 F 1 "16M" H 7850 2550 60  0000 C CNN
 F 2 "~" H 7850 2700 60  0000 C CNN
@@
 $EndComp
 $Comp
-L C C?
+L C C3
 U 1 1 531C7910
 P 8250 2400
-F 0 "C?" H 8250 2500 40  0000 L CNN
+F 0 "C3" H 8250 2500 40  0000 L CNN
 F 1 "27p" H 8256 2315 40  0000 L CNN
 F 2 "~" H 8288 2250 30  0000 C CNN
@@
 $EndComp
 $Comp
-L C C?
+L C C4
 U 1 1 531C791F
 P 8300 3000
-F 0 "C?" H 8300 3100 40  0000 L CNN
+F 0 "C4" H 8300 3100 40  0000 L CNN
 F 1 "27p" H 8306 2915 40  0000 L CNN
 F 2 "~" H 8338 2850 30  0000 C CNN
@@
 	3700 4450 3700 4600
 $Comp
-L R R?
+L R R3
 U 1 1 531C7BD5
 P 6350 3600
-F 0 "R?" V 6430 3600 40  0000 C CNN
+F 0 "R3" V 6430 3600 40  0000 C CNN
 F 1 "10k" V 6357 3601 40  0000 C CNN
 F 2 "~" V 6280 3600 30  0000 C CNN
@@
 	6600 3600 6800 3600
 $Comp
-L DIODE D?
+L DIODE D2
 U 1 1 531C9DEF
 P 1550 5950
-F 0 "D?" H 1550 6050 40  0000 C CNN
+F 0 "D2" H 1550 6050 40  0000 C CNN
 F 1 "1N4007" H 1550 5850 40  0000 C CNN
 F 2 "~" H 1550 5950 60  0000 C CNN
@@
 	1800 6000 1800 6300
 $Comp
-L NPN Q?
+L NPN Q1
 U 1 1 531CA881
 P 1700 6500
-F 0 "Q?" H 1700 6350 50  0000 R CNN
+F 0 "Q1" H 1700 6350 50  0000 R CNN
 F 1 "2N222" H 1700 6650 50  0000 R CNN
 F 2 "~" H 1700 6500 60  0000 C CNN
@@
 Connection ~ 1800 6150
 $Comp
-L R R?
+L R R1
 U 1 1 531CA8B2
 P 1200 6100
-F 0 "R?" V 1280 6100 40  0000 C CNN
+F 0 "R1" V 1280 6100 40  0000 C CNN
 F 1 "1K" V 1207 6101 40  0000 C CNN
 F 2 "~" V 1130 6100 30  0000 C CNN
@@
 $EndComp
 Wire Wire Line
-	1800 6700 1800 6850
-Wire Wire Line
 	1550 5750 1550 5650
 Text GLabel 1200 5700 1    60   Input ~ 0
@@
 	1200 6500 1500 6500
 $Comp
-L CONN_2 P?
+L CONN_2 P2
 U 1 1 531CABCB
 P 3100 5900
-F 0 "P?" V 3050 5900 40  0000 C CNN
+F 0 "P2" V 3050 5900 40  0000 C CNN
 F 1 "CONN_2" V 3150 5900 40  0000 C CNN
 F 2 "" H 3100 5900 60  0000 C CNN
@@
 	2750 6000 2750 6150
 $Comp
-L RELAY_1RT K?
+L RELAY_1RT K3
 U 1 1 531CB06A
 P 2200 5650
-F 0 "K?" H 2150 6050 70  0000 C CNN
+F 0 "K3" H 2150 6050 70  0000 C CNN
 F 1 "RELAY_1RT" H 2350 5150 70  0000 C CNN
 F 2 "~" H 2200 5650 60  0000 C CNN
@@
 	1550 5750 1800 5750
 $Comp
-L DIODE D?
+L DIODE D3
 U 1 1 531CB17E
 P 3800 5950
-F 0 "D?" H 3800 6050 40  0000 C CNN
+F 0 "D3" H 3800 6050 40  0000 C CNN
 F 1 "1N4007" H 3800 5850 40  0000 C CNN
 F 2 "~" H 3800 5950 60  0000 C CNN
@@
 	4050 6000 4050 6300
 $Comp
-L NPN Q?
+L NPN Q2
 U 1 1 531CB186
 P 3950 6500
-F 0 "Q?" H 3950 6350 50  0000 R CNN
+F 0 "Q2" H 3950 6350 50  0000 R CNN
 F 1 "2N222" H 3950 6650 50  0000 R CNN
 F 2 "~" H 3950 6500 60  0000 C CNN
@@
 Connection ~ 4050 6150
 $Comp
-L R R?
+L R R2
 U 1 1 531CB18D
 P 3450 6100
-F 0 "R?" V 3530 6100 40  0000 C CNN
+F 0 "R2" V 3530 6100 40  0000 C CNN
 F 1 "1K" V 3457 6101 40  0000 C CNN
 F 2 "~" V 3380 6100 30  0000 C CNN
@@
 $EndComp
 Wire Wire Line
-	4050 6700 4050 6850
-Wire Wire Line
 	3800 5750 3800 5650
 Text GLabel 3450 5700 1    60   Input ~ 0
 Light2
 Wire Wire Line
-	3450 5700 3450 5850
-Wire Wire Line
 	3450 6350 3450 6500
 Wire Wire Line
 	3450 6500 3750 6500
 $Comp
-L CONN_2 P?
+L CONN_2 P3
 U 1 1 531CB1A6
 P 5350 5900
-F 0 "P?" V 5300 5900 40  0000 C CNN
+F 0 "P3" V 5300 5900 40  0000 C CNN
 F 1 "CONN_2" V 5400 5900 40  0000 C CNN
 F 2 "" H 5350 5900 60  0000 C CNN
@@
 	5000 6000 5000 6150
 $Comp
-L RELAY_1RT K?
+L RELAY_1RT K4
 U 1 1 531CB1B4
 P 4450 5650
-F 0 "K?" H 4400 6050 70  0000 C CNN
+F 0 "K4" H 4400 6050 70  0000 C CNN
 F 1 "RELAY_1RT" H 4600 5150 70  0000 C CNN
 F 2 "~" H 4450 5650 60  0000 C CNN
@@
 $EndComp
 $Comp
-L CONN_2 P?
+L CONN_2 P1
 U 1 1 531CB273
 P 900 1850
-F 0 "P?" V 850 1850 40  0000 C CNN
+F 0 "P1" V 850 1850 40  0000 C CNN
 F 1 "CONN_2" V 950 1850 40  0000 C CNN
 F 2 "" H 900 1850 60  0000 C CNN
@@
 $EndComp
 Wire Wire Line
-	1250 1750 1450 1750
+	1250 1750 1650 1750
 Wire Wire Line
 	1450 1750 1450 1700
 Wire Wire Line
-	1250 1950 1450 1950
+	1250 1950 1650 1950
 Wire Wire Line
 	1450 1950 1450 2050
 $Comp
-L CONN_3 K?
+L CONN_3 K1
 U 1 1 531CB7C5
 P 900 2700
-F 0 "K?" V 850 2700 50  0000 C CNN
+F 0 "K1" V 850 2700 50  0000 C CNN
 F 1 "CONN_3" V 950 2700 40  0000 C CNN
 F 2 "" H 900 2700 60  0000 C CNN
@@
 $EndComp
 $Comp
-L GND #PWR?
+L GND #PWR017
 U 1 1 531CB7F6
 P 1400 2950
-F 0 "#PWR?" H 1400 2950 30  0001 C CNN
+F 0 "#PWR017" H 1400 2950 30  0001 C CNN
 F 1 "GND" H 1400 2880 30  0001 C CNN
 F 2 "" H 1400 2950 60  0000 C CNN
@@
 $EndComp
 $Comp
-L +5V #PWR?
+L +5V #PWR018
 U 1 1 531CB805
 P 1400 2550
-F 0 "#PWR?" H 1400 2640 20  0001 C CNN
+F 0 "#PWR018" H 1400 2640 20  0001 C CNN
 F 1 "+5V" H 1400 2640 30  0000 C CNN
 F 2 "" H 1400 2550 60  0000 C CNN
@@
 	1400 2800 1250 2800
 $Comp
-L CONN_3 K?
+L CONN_3 K2
 U 1 1 531CB8D3
 P 900 3500
-F 0 "K?" V 850 3500 50  0000 C CNN
+F 0 "K2" V 850 3500 50  0000 C CNN
 F 1 "CONN_3" V 950 3500 40  0000 C CNN
 F 2 "" H 900 3500 60  0000 C CNN
@@
 $EndComp
 $Comp
-L GND #PWR?
+L GND #PWR019
 U 1 1 531CB8D9
 P 1400 3750
-F 0 "#PWR?" H 1400 3750 30  0001 C CNN
+F 0 "#PWR019" H 1400 3750 30  0001 C CNN
 F 1 "GND" H 1400 3680 30  0001 C CNN
 F 2 "" H 1400 3750 60  0000 C CNN
@@
 $EndComp
 $Comp
-L +5V #PWR?
+L +5V #PWR020
 U 1 1 531CB8DF
 P 1400 3350
-F 0 "#PWR?" H 1400 3440 20  0001 C CNN
+F 0 "#PWR020" H 1400 3440 20  0001 C CNN
 F 1 "+5V" H 1400 3440 30  0000 C CNN
 F 2 "" H 1400 3350 60  0000 C CNN
@@
 Wire Wire Line
 	1400 3600 1250 3600
+Wire Wire Line
+	3450 5850 3450 5700
+Wire Wire Line
+	3850 2450 3850 2150
+Wire Wire Line
+	3850 2300 3700 2300
+Connection ~ 3850 2300
+$Comp
+L +5V #PWR021
+U 1 1 531CDB22
+P 3700 2000
+F 0 "#PWR021" H 3700 2090 20  0001 C CNN
+F 1 "+5V" H 3700 2090 30  0000 C CNN
+F 2 "" H 3700 2000 60  0000 C CNN
+F 3 "" H 3700 2000 60  0000 C CNN
+	1    3700 2000
+	1    0    0    -1
+$EndComp
+Wire Wire Line
+	3700 2300 3700 2000
+$Comp
+L PWR_FLAG #FLG022
+U 1 1 531CDC43
+P 1650 1750
+F 0 "#FLG022" H 1650 1845 30  0001 C CNN
+F 1 "PWR_FLAG" H 1650 1930 30  0000 C CNN
+F 2 "" H 1650 1750 60  0000 C CNN
+F 3 "" H 1650 1750 60  0000 C CNN
+	1    1650 1750
+	1    0    0    -1
+$EndComp
+Connection ~ 1450 1750
+Wire Wire Line
+	4050 6700 4050 6850
+Wire Wire Line
+	1800 6700 1800 6850
+$Comp
+L PWR_FLAG #FLG023
+U 1 1 531CDD98
+P 1650 1950
+F 0 "#FLG023" H 1650 2045 30  0001 C CNN
+F 1 "PWR_FLAG" H 1650 2130 30  0000 C CNN
+F 2 "" H 1650 1950 60  0000 C CNN
+F 3 "" H 1650 1950 60  0000 C CNN
+	1    1650 1950
+	-1   0    0    1
+$EndComp
+Connection ~ 1450 1950
 $EndSCHEMATC
